File: BasePower.kicad_sch (KiCad schematic)
At the start: 8 parts, among them U1 TPSM84203, U6 L7812

Commit message: minor fixes to power delivery
Parts:
- C31, C32: footprint (none) -> Capacitor_SMD:C_0805_2012Metric
Changed lines of the file:
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@@
 			)
 		)
-		(property "Footprint" ""
+		(property "Footprint" "Capacitor_SMD:C_0805_2012Metric"
 			(at 171.1452 127 0)
 			(effects
@@
 			)
 		)
-		(property "Footprint" ""
+		(property "Footprint" "Capacitor_SMD:C_0805_2012Metric"
 			(at 160.9852 127 0)
 			(effects
