File: power_switch.kicad_sch (KiCad schematic)
At the start: 15 parts, among them IC1 TMCS1123B1AQDVGR, IC2 LTC7067RMSE#PBF, IC3 LTC7067RMSE#PBF, J1 Conn_01x02_Socket, J2 Conn_01x02_Socket, Q1 NMOS, Q2 NMOS, Q3 NMOS, Q4 NMOS

Commit message: minor fixes to power delivery
Changed lines of the file:
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@@
 		)
 	)
-	(label "G2RTN"
+	(label "G4RTN"
 		(at 104.14 35.56 90)
 		(fields_autoplaced yes)
@@
 		)
 	)
-	(label "G1RTN"
+	(label "G3RTN"
 		(at 246.38 43.18 0)
 		(fields_autoplaced yes)
@@
 		)
 	)
-	(label "G2RTN"
+	(label "G3RTN"
 		(at 104.14 62.23 90)
 		(fields_autoplaced yes)
@@
 		)
 	)
-	(label "G2RTN"
+	(label "G4RTN"
 		(at 246.38 50.8 0)
 		(fields_autoplaced yes)
