File: Eload.kicad_sch (KiCad schematic)
At the start: 17 parts, among them J3 CAN, J5 Conn_01x03_Pin, J6 Conn_01x04_Pin, SW1 PTS820, SW3 RotaryEncoder_Switch

Commit message: minor fixes to power delivery
Parts:
- C2: footprint (none) -> Capacitor_SMD:C_0805_2012Metric
Changed lines of the file:
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@@
 			)
 		)
-		(property "Footprint" ""
+		(property "Footprint" "Capacitor_SMD:C_0805_2012Metric"
 			(at 103.8352 181.61 0)
 			(effects

Commit message: power switch stuff
Parts:
- SW3: footprint (none) -> Rotary_Encoder:RotaryEncoder_Alps_EC11E-Switch_Vertical_H20mm
Changed lines of the file:
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@@
 			)
 		)
-		(property "Footprint" ""
+		(property "Footprint" "Rotary_Encoder:RotaryEncoder_Alps_EC11E-Switch_Vertical_H20mm"
 			(at 226.06 98.806 0)
 			(effects
